File: PCB/CM4/connectors.sch (KiCad schematic (older format))
At the start: 12 parts, among them K1 CONN_3, K2 CONN_3, K3 CONN_3, K4 CONN_3, K5 CONN_3, K6 CONN_3, K7 CONN_3, K8 CONN_3, P1 CONN_2, U4 AP1115A

Commit message: 5v power  and reset
Parts:
- added C18: 10uF, symbol C
- added C19: 0.1uF, symbol C
- added D1: DIODE, symbol DIODE
- added SW1: SW_PUSH, symbol SW_PUSH
- added U5: LM7805, symbol LM7805
- renumbered C12 to C20, C13 to C21, U4 to U6
Connections:
- net +5V: now also U6.1 (V_IN), D1.2 (K)
- net +BATT: now also C18.1, U5.VI; no longer U6.1 (V_IN)
- net GND: now also C18.2, C19.2, SW1.1, U5.GND
- new net: D1.1 (A), U5.VO
- new net RESET: C19.1, SW1.2
Other:
- moved on the sheet: P1, U6
